File: eagle/GALI.brd (EAGLE design)
At the start: 60.9 x 180 mm, 114 parts, among them IC1 Z0103, IC10 Z0103, IC11 Z0103, IC12 Z0103, IC13 Z0103, IC14 Z0103, IC15 Z0103, IC16 Z0103, IC2 Z0103, IC3 Z0103, IC4 Z0103, IC5 Z0103, IC6 Z0103, IC7 Z0103, IC8 Z0103, IC9 Z0103

Commit message: Add files via upload
Parts:
- added AK18: AK130/02, ptr_ak130:AK02
- C1, C10, C11, C12, C13, C14, C15, C16, C2, C3, C4, C5, C6, C7, C8, C9: value (none) -> 0,1uFx250v
- R17, R19, R21, R23, R25, R27, R29, R31, R33, R35, R37, R39, R41, R43, R45, R47: value (none) -> 400
- R18, R20, R22, R24, R26, R28, R30, R32, R34, R36, R38, R40, R42, R44, R46, R48: value (none) -> 100
- moved AK16 746.5 mm to (170.2, 138.4), turned to 180 degrees
- moved AK14 710.7 mm to (170.2, 121.9), turned to 180 degrees
- moved AK17 709.4 mm to (16.5, 138.4)
- moved AK12 675.3 mm to (170.2, 105.4), turned to 180 degrees
- moved AK15 671.0 mm to (16.5, 121.9)
- moved AK10 640.4 mm to (170.2, 88.9), turned to 180 degrees
- moved AK13 632.7 mm to (16.5, 105.4)
- moved AK8 606.0 mm to (170.2, 72.4), turned to 180 degrees
- moved AK11 594.5 mm to (16.5, 88.9)
- moved AK6 572.3 mm to (170.2, 55.9), turned to 180 degrees
- moved IC15 561.8 mm to (127.0, 137.2), turned to 90 degrees
- moved AK9 556.5 mm to (16.5, 72.4)
- moved IC16 539.8 mm to (59.7, 139.7), turned to 270 degrees
- moved IC13 539.0 mm to (127.0, 120.7), turned to 90 degrees
- moved AK3 529.9 mm to (170.2, 39.4), turned to 180 degrees
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Connections:
- removed net N$115: AK4.2, AK5.2
- removed net N$50 (its old number): IC1.1, R17.2, R18.1
- removed net N$52 (its old number): IC2.1, R19.2, R20.1
- removed net N$54 (its old number): IC3.1, R21.2, R22.1
- removed net N$56 (its old number): IC4.1, R23.2, R24.1
- removed net N$58 (its old number): IC5.1, R25.2, R26.1
- removed net N$60 (its old number): IC6.1, R27.2, R28.1
- removed net N$62 (its old number): IC7.1, R29.2, R30.1
- removed net N$64 (its old number): IC8.1, R31.2, R32.1
- removed net N$66: IC9.1, R33.2, R34.1
- removed net N$70: IC11.1, R37.2, R38.1
- removed net N$72 (its old number): IC12.1, R39.2, R40.1
- removed net N$74 (its old number): IC13.1, R41.2, R42.1
- removed net N$76 (its old number): IC14.1, R43.2, R44.1
- removed net N$78 (its old number): IC15.1, R45.2, R46.1
- removed net N$80 (its old number): IC16.1, R47.2, R48.1
- new net N$112: AK11.2, AK13.2, AK15.2, AK17.2, AK18.1, AK18.2, AK2.2, AK4.2, AK7.2, AK9.2, IC10.1, IC12.1, IC14.1, IC16.1, IC2.1, IC4.1, IC6.1, IC8.1, R19.2, R20.1, R23.2, R24.1, R27.2, R28.1, R31.2, R32.1, R35.2, R36.1, R39.2, R40.1, R43.2, R44.1, R47.2, R48.1
- net N$68: now also AK1.2, AK10.2, AK12.2, AK14.2, AK16.2, AK3.2, AK5.1, AK5.2, AK6.2, AK8.2, IC1.1, IC11.1, IC13.1, IC15.1, IC3.1, IC5.1, IC7.1, IC9.1, R17.2, R18.1, R21.2, R22.1, R25.2, R26.1, R29.2, R30.1, R33.2, R34.1, R37.2, R38.1, R41.2, R42.1, R45.2, R46.1; no longer IC10.1, R35.2, R36.1
- net N$89: no longer AK5.1
Routing:
- net N$112: track 0.00 -> 591.2 mm
- net N$68: track 0.00 -> 588.4 mm
- net N$17: track 0.00 -> 428.5 mm
- net N$1: track 0.00 -> 71.1 mm
- net N$32: track 0.00 -> 68.6 mm
- net N$16: track 0.00 -> 59.7 mm
- net N$19: track 0.00 -> 57.1 mm
- net N$31: track 0.00 -> 54.6 mm
- net N$30: track 0.00 -> 54.6 mm
- net N$83: track 0.00 -> 49.6 mm
- net N$111: track 0.00 -> 47.3 mm
- net N$97: track 0.00 -> 47.3 mm
- net N$99: track 0.00 -> 47.3 mm
- net N$109: track 0.00 -> 47.3 mm
- net N$107: track 0.00 -> 47.3 mm
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Other:
- board size 60.9 x 180 mm -> 185.4 x 162.2 mm
