File: eagle/GALI.sch (EAGLE design)
At the start: 114 parts, among them IC1 Z0103, IC10 Z0103, IC11 Z0103, IC12 Z0103, IC13 Z0103, IC14 Z0103, IC15 Z0103, IC16 Z0103, IC2 Z0103, IC3 Z0103, IC4 Z0103, IC5 Z0103, IC6 Z0103, IC7 Z0103, IC8 Z0103, IC9 Z0103

Commit message: Add files via upload
Parts:
- added AK18: AK130/02, ptr_ak130:AK130/02
- C1, C10, C11, C12, C13, C14, C15, C16, C2, C3, C4, C5, C6, C7, C8, C9: value (none) -> 0,1uFx250v
- R17, R19, R21, R23, R25, R27, R29, R31, R33, R35, R37, R39, R41, R43, R45, R47: value (none) -> 400
- R18, R20, R22, R24, R26, R28, R30, R32, R34, R36, R38, R40, R42, R44, R46, R48: value (none) -> 100
Connections:
- removed net N$115: AK4.P$2, AK5.P$2
- removed net N$50 (its old number): IC1.C1, R17.2, R18.1
- removed net N$52 (its old number): IC2.C1, R19.2, R20.1
- removed net N$54 (its old number): IC3.C1, R21.2, R22.1
- removed net N$56 (its old number): IC4.C1, R23.2, R24.1
- removed net N$58 (its old number): IC5.C1, R25.2, R26.1
- removed net N$60 (its old number): IC6.C1, R27.2, R28.1
- removed net N$62 (its old number): IC7.C1, R29.2, R30.1
- removed net N$64 (its old number): IC8.C1, R31.2, R32.1
- removed net N$66: IC9.C1, R33.2, R34.1
- removed net N$70: IC11.C1, R37.2, R38.1
- removed net N$72 (its old number): IC12.C1, R39.2, R40.1
- removed net N$74 (its old number): IC13.C1, R41.2, R42.1
- removed net N$76 (its old number): IC14.C1, R43.2, R44.1
- removed net N$78 (its old number): IC15.C1, R45.2, R46.1
- removed net N$80 (its old number): IC16.C1, R47.2, R48.1
- new net N$112: AK11.P$2, AK13.P$2, AK15.P$2, AK17.P$2, AK18.P$1, AK18.P$2, AK2.P$2, AK4.P$2, AK7.P$2, AK9.P$2, IC10.C1, IC12.C1, IC14.C1, IC16.C1, IC2.C1, IC4.C1, IC6.C1, IC8.C1, R19.2, R20.1, R23.2, R24.1, R27.2, R28.1, R31.2, R32.1, R35.2, R36.1, R39.2, R40.1, R43.2, R44.1, R47.2, R48.1
- net N$68: now also AK1.P$2, AK10.P$2, AK12.P$2, AK14.P$2, AK16.P$2, AK3.P$2, AK5.P$1, AK5.P$2, AK6.P$2, AK8.P$2, IC1.C1, IC11.C1, IC13.C1, IC15.C1, IC3.C1, IC5.C1, IC7.C1, IC9.C1, R17.2, R18.1, R21.2, R22.1, R25.2, R26.1, R29.2, R30.1, R33.2, R34.1, R37.2, R38.1, R41.2, R42.1, R45.2, R46.1; no longer IC10.C1, R35.2, R36.1
- net N$89: no longer AK5.P$1
Other:
- moved on the sheet: AK5
