File: eagle/head procesing.brd (EAGLE design)
At the start: 160 x 100 mm, 60 parts, among them IC1 24LC256P, IC2 75176AP, IC3 SCT2026CSSG-1, IC4 SCT2026CSSG-1, IC5 SCT2026CSSG-1, IC6 SCT2026CSSG-1, IC7 SCT2026CSSG-1, IC8 SCT2026CSSG-1, J1 power, X1 DMX IN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

Commit message: Add files via upload
Parts:
- added C4: 47uFx35v, rcl:E2-5
- added C5: 0,47, cap-pan40:C5,0-7,5X3,5
- added IC9: LM2937ET-3.3, lm2937:TO220(V)
- added JP1, JP10, JP11, JP12, JP13, JP14, JP15, JP16, JP17, JP18, JP19, JP20, JP21, JP22, JP23, JP24, JP3, JP4, JP5, JP6, JP7, JP8, JP9: (no value), pinhead:1X01
- added R25, R26, R27: (no value), resistor:0207/10
- C10, C12, C14, C16, C3, C6, C7, C8: value (none) -> 0,1
- C2: value (none) -> o,1
- Q1: value (none) -> 5MHz
- R1, R11, R3, R5, R7, R9: value (none) -> 1k
- X1: device con-molex:KK-156-3 -> con-molex:70543-03
- moved R6 104.9 mm to (36.8, 71.1), turned to 180 degrees
- moved R4 97.0 mm to (36.8, 67.9)
- moved JP2 93.2 mm to (53.3, 68.6)
- moved SV5 71.8 mm to (116.8, 77.5), turned to 90 degrees
- moved R20 65.6 mm to (30.5, 11.4), turned to 270 degrees
- moved R12 63.1 mm to (35.6, 11.4), turned to 270 degrees
- moved C10 63.0 mm to (116.8, 49.5), flipped to the bottom, turned to 180 degrees
- moved IC7 62.7 mm to (116.8, 58.4), turned to 90 degrees
- moved R2 62.5 mm to (36.8, 35.6), turned to 90 degrees
- moved R5 62.0 mm to (116.8, 52.1), flipped to the bottom, turned to 180 degrees
- moved R10 59.6 mm to (33.0, 14.0), turned to 270 degrees
- moved SV2 58.3 mm to (80.0, 16.5), turned to 270 degrees
- moved R8 57.8 mm to (38.1, 14.0), turned to 270 degrees
- moved C16 52.8 mm to (116.8, 44.5), flipped to the bottom, turned to 0 degrees
- moved R11 48.3 mm to (116.8, 41.9), flipped to the bottom, turned to 0 degrees
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Connections:
- removed net N$146: INDICATE.6, R12.1, U$1.19
- removed net N$147: INDICATE.5, R10.1, U$1.18
- removed net N$148: INDICATE.4, R8.1, U$1.17
- removed net N$149: INDICATE.3, U$1.16
- removed net N$150: INDICATE.2, U$1.15
- removed net N$151: INDICATE.1, U$1.14
- removed net N$160: IC2.4, U$1.6
- removed net N$19: INDICATE.8, INDICATE.9
- removed net N$47: IC3.4, IC4.4, U$1.33
- removed net N$49: IC5.2, U$1.26
- removed net N$53: IC7.2, U$1.23
- removed net N$54: IC7.3, IC8.3, U$1.22
- removed net N$55: IC7.4, IC8.4, U$1.21
- new net CLK: INDICATE.8, U$1.14
- new net LA/: INDICATE.6, U$1.16
- new net N$16: IC3.3, IC4.3, JP3.1, JP4.1, U$1.34
- new net N$33: IC3.2, U$1.33
- new net N$36: IC3.4, IC4.4, JP1.1, JP5.1, U$1.35
- new net N$38: IC5.4, IC6.4, JP10.1, JP11.1, JP9.1, U$1.24
- new net N$6: IC2.3, R26.1, U$1.3
- new net S1-MENU: INDICATE.5, R8.1, U$1.17
- new net S2-UP: INDICATE.4, R10.1, U$1.18
- new net S3-DOWN: INDICATE.3, R12.1, U$1.19
- new net S4-ENTER: INDICATE.2, R20.1, U$1.20
- new net SDI: INDICATE.7, U$1.15
- net +3V3: now also C4.+, IC9.OUT, JP6.1, R10.2, R12.2, R20.2, R8.2; no longer J1.3
- net +5V: now also C5.2, IC9.IN, INDICATE.9, J1.3, JP7.1, JP8.1; no longer INDICATE.10
- net GND: now also C4.-, C5.1, IC9.GND, INDICATE.1, INDICATE.10, R25.2, R26.2, R27.2, U$1.10; no longer R10.2, R12.2, R20.2, R8.2
- net N$1: now also U$1.7; no longer U$1.3
- net N$145: now also IC7.4, IC8.4, JP18.1, JP19.1, JP20.1, U$1.21; no longer INDICATE.7, R20.1, U$1.20
- net N$158: now also R27.1, U$1.2; no longer U$1.5
- net N$159: now also IC2.4, R25.1, U$1.4; no longer IC2.3, U$1.7
- net N$2: now also U$1.6; no longer U$1.2
- net N$22: now also U$1.1; no longer U$1.4
- net N$3: now also U$1.5; no longer U$1.1
- net N$45: now also IC5.3, IC6.3, JP12.1, JP13.1, JP14.1, U$1.25; no longer IC3.2, U$1.35
- net N$46: now also IC5.2, JP16.1, JP17.1, U$1.26; no longer IC3.3, IC4.3, U$1.34
- net N$50: now also IC7.2, JP15.1, JP21.1, U$1.23; no longer IC5.3, IC6.3, U$1.25
- net N$51: now also IC7.3, IC8.3, JP22.1, JP23.1, JP24.1, U$1.22; no longer IC5.4, IC6.4, U$1.24
Routing:
- net +5V: track 0.00 -> 605.8 mm, vias 0 -> 1
- net GND: track 0.00 -> 510.3 mm
- net +3V3: track 0.00 -> 207.1 mm
- net N$51: track 0.00 -> 124.3 mm, vias 0 -> 1
- net N$145: track 0.00 -> 123.6 mm
- net N$38: track 0.00 -> 93.7 mm
- net N$45: track 0.00 -> 92.3 mm
- net N$50: track 0.00 -> 79.9 mm
- net N$36: track 0.00 -> 62.6 mm
- net N$9: track 0.00 -> 59.8 mm
- net N$16: track 0.00 -> 54.4 mm
- net N$46: track 0.00 -> 53.9 mm
- net N$158: track 0.00 -> 47.5 mm
- net N$144: track 0.00 -> 42.7 mm
- net N$6: track 0.00 -> 41.0 mm
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Other:
- board size 160 x 100 mm -> 130.8 x 94.3 mm
