File: eagle/head procesing.sch (EAGLE design)
At the start: 60 parts, among them IC1 24LC256P, IC2 75176AP, IC3 SCT2026CSSG-1, IC4 SCT2026CSSG-1, IC5 SCT2026CSSG-1, IC6 SCT2026CSSG-1, IC7 SCT2026CSSG-1, IC8 SCT2026CSSG-1, J1 power, X1 DMX IN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

Commit message: Add files via upload
Parts:
- added C4: 47uFx35v, rcl:CPOL-EUE2-5
- added C5: 0,47, cap-pan40:C-NP-5,0-7,5X3,5
- added IC9: LM2937ET-3.3, lm2937:LM2937ET-3.3
- added JP1, JP10, JP11, JP12, JP13, JP14, JP15, JP16, JP17, JP18, JP19, JP20, JP21, JP22, JP23, JP24, JP3, JP4, JP5, JP6, JP7, JP8, JP9: (no value), pinhead:PINHD-1X1
- added R25, R26, R27: (no value), resistor:R-US_0207/10
- C10, C12, C14, C16, C3, C6, C7, C8: value (none) -> 0,1
- C2: value (none) -> o,1
- Q1: value (none) -> 5MHz
- R1, R11, R3, R5, R7, R9: value (none) -> 1k
- X1: device con-molex:KK-156-3 -> con-molex:C-GRID-03-70543
Connections:
- removed net N$146: INDICATE-6.KL, R12.1, U$1P8X32A-D40.P14
- removed net N$147: INDICATE-5.KL, R10.1, U$1P8X32A-D40.P13
- removed net N$148: INDICATE-4.KL, R8.1, U$1P8X32A-D40.P12
- removed net N$149: INDICATE-3.KL, U$1P8X32A-D40.P11
- removed net N$150: INDICATE-2.KL, U$1P8X32A-D40.P10
- removed net N$151: INDICATE-1.KL, U$1P8X32A-D40.P9
- removed net N$160: IC2.D, U$1P8X32A-D40.P5
- removed net N$19: INDICATE-8.KL, INDICATE-9.KL
- removed net N$47: IC3.LA/, IC4.LA/, U$1P8X32A-D40.P24
- removed net N$49: IC5.SDI, U$1P8X32A-D40.P21
- removed net N$53: IC7.SDI, U$1P8X32A-D40.P18
- removed net N$54: IC7.CLK, IC8.CLK, U$1P8X32A-D40.P17
- removed net N$55: IC7.LA/, IC8.LA/, U$1P8X32A-D40.P16
- new net CLK: INDICATE-8.KL, U$1P8X32A-D40.P9
- new net LA/: INDICATE-6.KL, U$1P8X32A-D40.P11
- new net N$16: IC3.CLK, IC4.CLK, JP3.1, JP4.1, U$1P8X32A-D40.P25
- new net N$33: IC3.SDI, U$1P8X32A-D40.P24
- new net N$36: IC3.LA/, IC4.LA/, JP1.1, JP5.1, U$1P8X32A-D40.P26
- new net N$38: IC5.LA/, IC6.LA/, JP10.1, JP11.1, JP9.1, U$1P8X32A-D40.P19
- new net N$6: IC2.DE, R26.1, U$1P8X32A-D40.P2
- new net S1-MENU: INDICATE-5.KL, R8.1, U$1P8X32A-D40.P12
- new net S2-UP: INDICATE-4.KL, R10.1, U$1P8X32A-D40.P13
- new net S3-DOWN: INDICATE-3.KL, R12.1, U$1P8X32A-D40.P14
- new net S4-ENTER: INDICATE-2.KL, R20.1, U$1P8X32A-D40.P15
- new net SDI: INDICATE-7.KL, U$1P8X32A-D40.P10
- net +3V3: now also C4.+, IC9.OUT, JP6.1, R10.2, R12.2, R20.2, R8.2; no longer J1.3
- net +5V: now also C5.2, IC9.IN, INDICATE-9.KL, J1.3, JP7.1, JP8.1; no longer INDICATE-10.KL
- net GND: now also C4.-, C5.1, IC9.GND, INDICATE-1.KL, INDICATE-10.KL, R25.2, R26.2, R27.2, U$1P8X32A-D40.BOE/; no longer R10.2, R12.2, R20.2, R8.2
- net N$1: now also U$1P8X32A-D40.P6; no longer U$1P8X32A-D40.P2
- net N$145: now also IC7.LA/, IC8.LA/, JP18.1, JP19.1, JP20.1, U$1P8X32A-D40.P16; no longer INDICATE-7.KL, R20.1, U$1P8X32A-D40.P15
- net N$158: now also R27.1, U$1P8X32A-D40.P1; no longer U$1P8X32A-D40.P4
- net N$159: now also IC2.D, R25.1, U$1P8X32A-D40.P3; no longer IC2.DE, U$1P8X32A-D40.P6
- net N$2: now also U$1P8X32A-D40.P5; no longer U$1P8X32A-D40.P1
- net N$22: now also U$1P8X32A-D40.P0; no longer U$1P8X32A-D40.P3
- net N$3: now also U$1P8X32A-D40.P4; no longer U$1P8X32A-D40.P0
- net N$45: now also IC5.CLK, IC6.CLK, JP12.1, JP13.1, JP14.1, U$1P8X32A-D40.P20; no longer IC3.SDI, U$1P8X32A-D40.P26
- net N$46: now also IC5.SDI, JP16.1, JP17.1, U$1P8X32A-D40.P21; no longer IC3.CLK, IC4.CLK, U$1P8X32A-D40.P25
- net N$50: now also IC7.SDI, JP15.1, JP21.1, U$1P8X32A-D40.P18; no longer IC5.CLK, IC6.CLK, U$1P8X32A-D40.P20
- net N$51: now also IC7.CLK, IC8.CLK, JP22.1, JP23.1, JP24.1, U$1P8X32A-D40.P17; no longer IC5.LA/, IC6.LA/, U$1P8X32A-D40.P19
Other:
- moved on the sheet: INDICATE-1, INDICATE-10, INDICATE-2, INDICATE-3, INDICATE-4, INDICATE-5, INDICATE-6, INDICATE-7, INDICATE-8, INDICATE-9, J1
