File: eagle/indicate switch.sch (EAGLE design)
At the start: 13 parts, among them IC1 SCT2026CSSG-1, IC2 SCT2026CSSG-1

Commit message: Add files via upload
Connections:
- removed net N$7: C1.1, C2.1, IC1.GND, IC2.GND, R1.1, R2.1, SV1-9.S
- net N$1: now also S2.2; no longer S1.2
- net N$12: now also S3.2, SV1-3.S; no longer IC1.SDI, SV1-1.S
- net N$13: now also SV1-8.S; no longer SV1-2.S
- net N$14: now also SV1-6.S; no longer SV1-3.S
- net N$19: now also DIS1.D2
- net N$2: now also S1.2; no longer S2.2
- net N$3: now also S4.2, SV1-2.S; no longer S3.2, SV1-6.S
- net N$4: now also IC1.SDI; no longer S4.2
- net N$5: now also C1.1, C2.1, IC1.GND, IC2.GND, R1.1, R2.1, SV1-1.S, SV1-10.S; no longer SV1-8.S
- net N$6: now also SV1-9.S; no longer SV1-10.S
Other:
- moved on the sheet: SV1-1, SV1-10, SV1-2, SV1-3, SV1-4, SV1-5, SV1-6, SV1-7, SV1-8, SV1-9
